File: Week 2/KiCAD Assignment/Assignment.kicad_sch (KiCad schematic)
At the start: 10 parts, among them J1 USB_C_Receptacle_PowerOnly_6P, J2 Conn_01x02_Pin

Commit message: Ruchika_Kicad assignment
Parts:
- C1, C2: footprint (none) -> Capacitor_SMD:C_1206_3216Metric_Pad1.33x1.80mm_HandSolder
- D1, D2: footprint (none) -> LED_THT:LED_D3.0mm
- J1: footprint (none) -> Connector_USB:USB_C_Receptacle_GCT_USB4125-xx-x-0190_6P_TopMnt_Horizontal
- J2: footprint (none) -> Connector_PinHeader_1.00mm:PinHeader_1x02_P1.00mm_Vertical_SMD_Pin1Left
- R1, R2, R3: footprint (none) -> Resistor_SMD:R_0805_2012Metric_Pad1.20x1.40mm_HandSolder
- TP1: footprint (none) -> Package_SO:SOP-8_5.28x5.23mm_P1.27mm
Connections:
- net at R2.2: now also TP1.6 (STDBY); no longer TP1.5 (STDBY)
Other:
- moved on the sheet: J2
Changed lines of the file:
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@@
+	(wire
+		(pts
+			(xy 142.24 31.75) (xy 228.6 31.75)
+		)
+		(stroke
+			(width 0)
+			(type default)
+		)
+	)
+	(wire
+		(pts
+			(xy 116.84 64.77) (xy 106.68 64.77)
+		)
+		(stroke
+			(width 0)
+			(type default)
+		)
+	)
+	(wire
+		(pts
+			(xy 161.29 81.28) (xy 161.29 80.01)
+		)
+		(stroke
+			(width 0)
+			(type default)
+		)
+	)
+	(wire
+		(pts
+			(xy 133.35 64.77) (xy 133.35 69.85)
+		)
+		(stroke
+			(width 0)
+			(type default)
+		)
+	)
+	(wire
+		(pts
+			(xy 116.84 93.98) (xy 133.35 93.98)
+		)
+		(stroke
+			(width 0)
+			(type default)
+		)
+	)
+	(wire
+		(pts
+			(xy 224.79 45.72) (xy 228.6 45.72)
+		)
+		(stroke
+			(width 0)
+			(type default)
+		)
+	)
+	(wire
+		(pts
+			(xy 180.34 90.17) (xy 236.22 90.17)
+		)
+		(stroke
+			(width 0)
+			(type default)
+		)
+	)
 	(wire
 		(pts
@@
 	(wire
 		(pts
-			(xy 116.84 64.77) (xy 106.68 64.77)
-		)
-		(stroke
-			(width 0)
-			(type default)
-		)
-	)
-	(wire
-		(pts
-			(xy 161.29 81.28) (xy 161.29 80.01)
-		)
-		(stroke
-			(width 0)
-			(type default)
-		)
-	)
-	(wire
-		(pts
-			(xy 133.35 64.77) (xy 133.35 69.85)
-		)
-		(stroke
-			(width 0)
-			(type default)
-		)
-	)
-	(wire
-		(pts
-			(xy 116.84 93.98) (xy 133.35 93.98)
-		)
-		(stroke
-			(width 0)
-			(type default)
-		)
-	)
-	(wire
-		(pts
-			(xy 224.79 45.72) (xy 228.6 45.72)
+			(xy 236.22 90.17) (xy 236.22 100.33)
+		)
+		(stroke
+			(width 0)
+			(type default)
+		)
+	)
+	(wire
+		(pts
+			(xy 172.72 64.77) (xy 180.34 64.77)
 		)
 		(stroke
@@
 	(wire
 		(pts
-			(xy 236.22 101.6) (xy 227.33 101.6)
+			(xy 236.22 101.6) (xy 224.79 101.6)
 		)
 		(stroke
@@
 	(wire
 		(pts
+			(xy 228.6 31.75) (xy 228.6 40.64)
+		)
+		(stroke
+			(width 0)
+			(type default)
+		)
+	)
+	(wire
+		(pts
 			(xy 133.35 73.66) (xy 125.73 73.66)
 		)
@@
 	(wire
 		(pts
+			(xy 142.24 57.15) (xy 142.24 31.75)
+		)
+		(stroke
+			(width 0)
+			(type default)
+		)
+	)
+	(wire
+		(pts
 			(xy 172.72 69.85) (xy 165.1 69.85)
 		)
@@
 	(wire
 		(pts
-			(xy 236.22 104.14) (xy 227.33 104.14)
+			(xy 236.22 104.14) (xy 224.79 104.14)
 		)
 		(stroke
@@
 	(wire
 		(pts
+			(xy 180.34 64.77) (xy 180.34 90.17)
+		)
+		(stroke
+			(width 0)
+			(type default)
+		)
+	)
+	(wire
+		(pts
 			(xy 142.24 64.77) (xy 133.35 64.77)
 		)
@@
 	(wire
 		(pts
-			(xy 236.22 105.41) (xy 236.22 104.14)
+			(xy 236.22 104.14) (xy 236.22 105.41)
 		)
 		(stroke
@@
 		(on_board yes)
 		(dnp no)
-		(fields_autoplaced yes)
 		(property "Reference" "#PWR09"
 			(at 172.72 71.12 0)
@@
 		)
 		(property "Value" "VD"
-			(at 172.72 62.23 0)
+			(at 173.228 62.738 0)
 			(effects
 				(font
@@
 			)
 		)
-		(property "Footprint" ""
+		(property "Footprint" "LED_THT:LED_D3.0mm"
 			(at 125.73 77.47 0)
 			(effects
@@
 			)
 		)
-		(property "Footprint" ""
+		(property "Footprint" "Resistor_SMD:R_0805_2012Metric_Pad1.20x1.40mm_HandSolder"
 			(at 149.352 86.36 90)
 			(effects
@@
 	(symbol
 		(lib_id "Connector:Conn_01x02_Pin")
-		(at 222.25 101.6 0)
+		(at 219.71 101.6 0)
 		(unit 1)
 		(exclude_from_sim no)
@@
 		(fields_autoplaced yes)
 		(property "Reference" "J2"
-			(at 222.885 96.52 0)
+			(at 220.345 96.52 0)
 			(effects
 				(font
@@
 		)
 		(property "Value" "Conn_01x02_Pin"
-			(at 222.885 99.06 0)
-			(effects
-				(font
-					(size 1.27 1.27)
-				)
-			)
-		)
-		(property "Footprint" ""
-			(at 222.25 101.6 0)
+			(at 220.345 99.06 0)
+			(effects
+				(font
+					(size 1.27 1.27)
+				)
+			)
+		)
+		(property "Footprint" "Connector_PinHeader_1.00mm:PinHeader_1x02_P1.00mm_Vertical_SMD_Pin1Left"
+			(at 219.71 101.6 0)
 			(effects
 				(font
@@
 		)
 		(property "Datasheet" "~"
-			(at 222.25 101.6 0)
+			(at 219.71 101.6 0)
 			(effects
 				(font
@@
 		)
 		(property "Description" "Generic connector, single row, 01x02, script generated"
-			(at 222.25 101.6 0)
+			(at 219.71 101.6 0)
 			(effects
 				(font
@@
 			)
 		)
-		(property "Footprint" ""
+		(property "Footprint" "Resistor_SMD:R_0805_2012Metric_Pad1.20x1.40mm_HandSolder"
 			(at 123.952 85.09 90)
 			(effects
@@
 			)
 		)
-		(property "Footprint" ""
+		(property "Footprint" "Capacitor_SMD:C_1206_3216Metric_Pad1.33x1.80mm_HandSolder"
 			(at 107.6452 78.74 0)
 			(effects
@@
 			)
 		)
-		(property "Footprint" ""
+		(property "Footprint" "Package_SO:SOP-8_5.28x5.23mm_P1.27mm"
 			(at 142.24 77.47 0)
 			(effects
@@
 		(pin "1"
 		)
-		(pin ""
-		)
-		(pin "5"
+		(pin "6"
 		)
 		(pin "2"
@@
 			)
 		)
-		(property "Footprint" ""
+		(property "Footprint" "LED_THT:LED_D3.0mm"
 			(at 116.84 77.47 0)
 			(effects
@@
 			)
 		)
-		(property "Footprint" ""
+		(property "Footprint" "Connector_USB:USB_C_Receptacle_GCT_USB4125-xx-x-0190_6P_TopMnt_Horizontal"
 			(at 213.36 50.8 0)
 			(effects
@@
 			)
 		)
-		(property "Footprint" ""
+		(property "Footprint" "Resistor_SMD:R_0805_2012Metric_Pad1.20x1.40mm_HandSolder"
 			(at 115.062 85.09 90)
 			(effects
@@
 			)
 		)
-		(property "Footprint" ""
+		(property "Footprint" "Capacitor_SMD:C_1206_3216Metric_Pad1.33x1.80mm_HandSolder"
 			(at 166.0652 77.47 0)
 			(effects
